Commit message: Flip the dependency between base_link and base_footprint

File: scarab_description/urdf/kobuki.urdf.xacro (robot description, xacro)
@@ -19,7 +19,7 @@
     -->
     <joint name="base_joint" type="fixed">
-      <origin xyz="0 0 0.0102" rpy="0 0 0" />
-      <parent link="base_footprint"/>
-      <child link="base_link" />
+      <origin xyz="0 0 -0.0102" rpy="0 0 0" />
+      <parent link="base_link" />
+      <child link="base_footprint"/>
     </joint>
     <link name="base_link">
